Commit message: first commit

File: bumperbot_description/urdf/bumperbot.urdf.xacro (robot description, xacro)
@@ -21,4 +21,7 @@
         <mesh filename="package://bumperbot_description/meshes/base_link.STL" />
       </geometry>
+      <material name="blue">
+        <color rgba="0.2 0.2 1 1"/>
+       </material>
     </visual>
     <collision>

File: bumperbot_description/urdf/bumperbot_gazebo.xacro (robot description, xacro)
@@ -1,5 +1,27 @@
 <?xml version="1.0"?>
 <robot name="bumperbot" xmlns:xacro="http://ros.org/wiki/xacro">
+ <!-- <material name="white">
+        <color rgba="1 1 1 1" />
+    </material>
+     <material name="red">
+        <color rgba="1 0 0 1" />
+    </material>
+    <material name="orange">
+        <color rgba="1 0.3 0.1 1"/>
+    </material>
+    <material name="blue">
+        <color rgba="0.2 0.2 1 1"/>
+    </material>
+    <material name="black">
+        <color rgba="0 0 0 1"/>
+    </material> -->
+    <xacro:property name="body_color_blue" value="Gazebo/Blue"/>
+   <!-- <gazebo reference="base_link">
+    <material>Gazebo/Blue</material>
+   </gazebo> -->
     <gazebo reference = "wheel_right_link">
+        <material>
+            Gazebo/Blue
+        </material>
         <mu1>100000000000000.0</mu1>
         <mu2>100000000000000.0</mu2>
@@ -11,4 +33,7 @@
     </gazebo>
     <gazebo reference = "wheel_left_link">
+        <material>
+            Gazebo/Blue
+        </material>
         <mu1>100000000000000.0</mu1>
         <mu2>100000000000000.0</mu2>
@@ -20,4 +45,7 @@
     </gazebo>
     <gazebo reference = "caster_front_link">
+        <material>
+            Gazebo/Black
+        </material>
         <mu1>0.1</mu1>
         <mu2>0.1</mu2>
@@ -28,4 +56,7 @@
     </gazebo>
     <gazebo reference = "caster_rear_link">
+        <material>
+            Gazebo/Black
+        </material>
         <mu1>0.1</mu1>
         <mu2>0.1</mu2>
@@ -59,5 +90,5 @@
         <topic>imu</topic>
         <imu>
-            <angular_velocity>
+            <!-- <angular_velocity>
                 <x>
                     <noise type="gaussian">
@@ -98,5 +129,5 @@
                     </noise>
                 </z>
-            </linear_acceleration>
+            </linear_acceleration> -->
         </imu>
         </sensor>
